Commit message: fix: update wrist camera gripper quality notes and compatibility docs

File: gbt-c5a_wrist_camera_gripper/urdf/gbt-c5a_wrist_camera_gripper.urdf (robot description, URDF)
Before this commit: robot GBT_C5A_wrist_camera_gripper, 21 links, 20 joints
Links:
- link base_link: mass 9.16039502558691 -> 1.489536
- link link1: mass 15.175 -> 4.763058
- link link2: mass 45.747 -> 10.922830
- link link3: mass 25.388 -> 3.817807
- link link4: mass 5.9625 -> 1.860492
- link link5: mass 6.3692 -> 1.823601
- link link6: mass 1.0139 -> 0.240531

Commit message: Fix camera_mount_joint rotation values

File: gbt-c5a_wrist_camera_gripper/urdf/gbt-c5a_wrist_camera_gripper.urdf (robot description, URDF)
Before this commit: robot GBT_C5A_wrist_camera_gripper, 21 links, 20 joints
Joints:
- joint camera_mount_joint: origin xyz=0 0 0.012 rpy=1.57079632679 0 3.1415926535 -> xyz=0 0 0.012 rpy=1.57079632679 0 0
